File: Labs/Lab8/EagleProject/HRM/HRM.sch (EAGLE design)
At the start: 14 parts, among them IC1 UA741P, IC2 UA741P, IC3 UA741P, J1 POWER_JACK, U1 QRD1114

Commit message: update from work in NXP lab
Parts:
- removed J1: POWER_JACK, SparkFun-Connectors:POWER_JACK
- added JP1: (no value), SparkFun-Connectors:M03PTH
- C1, C2: device SparkFun-Capacitors:1000UF-RADIAL-5MM-25V-20% -> resistor:C-USC3216
- R1, R2, R4, R5, R6, R7: device SparkFun-Resistors:RESISTORAXIAL-0.3 -> resistor:R-US_M1206
- R3: value (none) -> 57.3k; device SparkFun-Resistors:RESISTORAXIAL-0.3 -> resistor:R-US_M1206
Connections:
- removed net N$10: IC3.OUT, R6.2
- new net OUT: IC3.OUT, JP1.1, R6.1
- net +5V: now also JP1.3; no longer J1.PWR
- net GND: now also C2.2, JP1.2, R3.1, R7.2; no longer C2.-, J1.GND, J1.GNDBREAK, R3.2, R7.1
- net N$3: now also IC2.-IN
- net N$4: now also C1.1; no longer C1.+
- net N$5: now also C1.2, R3.2; no longer C1.-, R3.1
- net N$6: now also R5.2; no longer R5.1
- net N$7: now also C2.1, R5.1; no longer C2.+, R5.2
- net N$8: now also R6.2, R7.1; no longer R6.1, R7.2
Other:
- note added: "+5V"
- note added: "GND"
- note added: "OUT"
- moved on the sheet: R3, R5, R6, R7
